File: schematics/kicad/atx-mod-ctrl/atx-mod-ctrl.sch (KiCad schematic (older format))
At the start: 1 part

Commit message: Intermediate version
Parts:
- added C1, C2: 68n, Capacitor_THT:C_Rect_L4.0mm_W2.5mm_P2.50mm, symbol Device:C
- added D1, D2: 1N4148, Diode_THT:D_DO-35_SOD27_P7.62mm_Horizontal, symbol Diode:1N4148
- added D3: LED, symbol Device:LED
- added Q1: BC557, Package_TO_SOT_THT:TO-92_Inline, symbol Transistor_BJT:BC557
- added R1: 1.5k, Resistor_THT:R_Axial_DIN0207_L6.3mm_D2.5mm_P2.54mm_Vertical, symbol Device:R
- added R2: 10k, Resistor_THT:R_Axial_DIN0207_L6.3mm_D2.5mm_P2.54mm_Vertical, symbol Device:R
- added U2: LM358, symbol Amplifier_Operational:LM358
- gave numbers to parts that had none: 1
Connections:
- net labels added: GND, VREF, Vout
- wire segments 0 -> 39
Other:
- note added: "Limit voltage on COMP input \nto limit maximum PWM duty cycle"
- moved on the sheet: U1

Commit message: minor updates
Connections:
- wire segments 39 -> 45
Changed lines of the file:
@@
 	8450 2800 8450 1750
 Wire Wire Line
-	8450 1750 4350 1750
+	8450 1750 6250 1750
 $Comp
 L Device:R R2
@@
 Text Notes 4500 4600 0    50   ~ 0
 Limit voltage on COMP input \nto limit maximum PWM duty cycle
+Wire Wire Line
+	6500 2800 6250 2800
+Wire Wire Line
+	6250 2800 6250 1750
+Connection ~ 6250 1750
+Wire Wire Line
+	6250 1750 4350 1750
+Wire Wire Line
+	6500 3100 6250 3100
+Wire Wire Line
+	6250 3100 6250 3200
+Wire Wire Line
+	6250 3200 6500 3200
+$Comp
+L power:GND #PWR?
+U 1 1 5D627AD3
+P 6250 3200
+F 0 "#PWR?" H 6250 2950 50  0001 C CNN
+F 1 "GND" H 6255 3027 50  0000 C CNN
+F 2 "" H 6250 3200 50  0001 C CNN
+F 3 "" H 6250 3200 50  0001 C CNN
+	1    6250 3200
+	1    0    0    -1
+$EndComp
+Connection ~ 6250 3200
 $EndSCHEMATC
